Commit message: change the default

File: src/robots/lite3_description/urdf/lite3.urdf (robot description, URDF)
Before this commit: robot Lite3, 18 links, 17 joints
Joints:
- joint FL_HipX_joint: axis -1 0 0 -> 1 0 0
- joint FL_HipY_joint: axis 0 -1 0 -> 0 1 0; limit lower=-2.67 upper=0.314 effort=24 velocity=26.2 -> lower=-0.314 upper=2.67 effort=24 velocity=26.2
- joint FL_Knee_joint: axis 0 -1 0 -> 0 1 0; limit lower=0.524 upper=2.792 effort=36 velocity=17.3 -> lower=-2.792 upper=-0.524 effort=36 velocity=17.3
- joint FR_HipX_joint: axis -1 0 0 -> 1 0 0
- joint FR_HipY_joint: axis 0 -1 0 -> 0 1 0; limit lower=-2.67 upper=0.314 effort=24 velocity=26.2 -> lower=-0.314 upper=2.67 effort=24 velocity=26.2
- joint FR_Knee_joint: axis 0 -1 0 -> 0 1 0; limit lower=0.524 upper=2.792 effort=36 velocity=17.3 -> lower=-2.792 upper=-0.524 effort=36 velocity=17.3
- joint HL_HipX_joint: axis -1 0 0 -> 1 0 0
- joint HL_HipY_joint: axis 0 -1 0 -> 0 1 0; limit lower=-2.67 upper=0.314 effort=24 velocity=26.2 -> lower=-0.314 upper=2.67 effort=24 velocity=26.2
- joint HL_Knee_joint: axis 0 -1 0 -> 0 1 0; limit lower=0.524 upper=2.792 effort=36 velocity=17.3 -> lower=-2.792 upper=-0.524 effort=36 velocity=17.3
- joint HR_HipX_joint: axis -1 0 0 -> 1 0 0
- joint HR_HipY_joint: axis 0 -1 0 -> 0 1 0; limit lower=-2.67 upper=0.314 effort=24 velocity=26.2 -> lower=-0.314 upper=2.67 effort=24 velocity=26.2
- joint HR_Knee_joint: axis 0 -1 0 -> 0 1 0; limit lower=0.524 upper=2.792 effort=36 velocity=17.3 -> lower=-2.792 upper=-0.524 effort=36 velocity=17.3
